File: kicad/spellcaster.kicad_pcb (KiCad board)
At the start: 4 copper layers, 38 parts, among them SW1 SW_Push, SW2 SW_Push, U1 nRF52820-QDxx, Y1 32k, Y2 Crystal_GND24

Commit message: Initial routing
Parts:
- removed H3, H4: MountingHole, MountingHole:MountingHole_2.2mm_M2_Pad_Via
- removed SW1, SW2: SW_Push, Button_Switch_SMD:SW_SPST_PTS645
- added C14: 100n, Capacitor_SMD:C_0402_1005Metric, F.Cu at (55.2, 116.3)
- added C16: 100n, Capacitor_SMD:C_0402_1005Metric, F.Cu at (57.1, 116.3)
- added R2: 10k, Resistor_SMD:R_0402_1005Metric, F.Cu at (56.0, 111.3)
- added R3: 10k, Resistor_SMD:R_0402_1005Metric, F.Cu at (56.0, 112.3)
- added S2: B3U-1000P, Snapeda:SW_B3U-1000P, F.Cu at (54.7, 129.5)
- added U2: LSM6DSL, Package_LGA:LGA-14_3x2.5mm_P0.5mm_LayoutBorder3x4y, F.Cu at (56.1, 114.3)
- BT1: footprint Battery:BatteryHolder_Keystone_3002_1x2032 -> Connector_Wire:SolderWire-0.5sqmm_1x02_P4.8mm_D0.9mm_OD2.3mm
- moved BT1 107.1 mm to (52.7, 137.2)
- moved H2 106.4 mm to (69.5, 138.7)
- moved C2 72.1 mm to (51.7, 115.6), turned to 90 degrees
- moved C3 69.9 mm to (52.7, 115.6), turned to -90 degrees
- moved C1 68.7 mm to (53.4, 110.6)
- moved U1 66.8 mm to (55.0, 106.4), turned to 45 degrees
- moved S1 66.8 mm to (54.7, 119.1), turned to 180 degrees
- moved Y1 63.9 mm to (52.3, 113.4)
- moved C9 63.5 mm to (50.5, 108.0), turned to -90 degrees
- moved L4 62.2 mm to (51.3, 101.3), turned to 90 degrees
- moved C5 62.1 mm to (50.8, 110.0), turned to 90 degrees
- moved C12 61.8 mm to (53.5, 102.1), turned to 180 degrees
- moved C11 60.7 mm to (56.0, 100.3), turned to -90 degrees
- moved C7 59.7 mm to (58.7, 103.9), turned to 180 degrees
- moved C10 59.0 mm to (58.9, 109.1), turned to -90 degrees
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Connections:
- U1 pad 14: unconnected-(U1-P0.14-Pad14) -> SDA
- U1 pad 15: unconnected-(U1-P0.15-Pad15) -> SCL
- U1 pad 36: BTN_B -> unconnected-(U1-AIN0/P0.02-Pad36)
- U1 pad 6: unconnected-(U1-P0.06-Pad6) -> INT2
- U1 pad 7: GPIO -> INT1
Routing:
- net RST: track 0.00 -> 34.8 mm, vias 0 -> 4
- net SWDIO: track 0.00 -> 29.3 mm, vias 0 -> 2
- net BTN_A: track 0.00 -> 29.1 mm, vias 0 -> 2
- net SWDCLK: track 0.00 -> 25.9 mm, vias 0 -> 2
- net Net-(U1-DEC4): track 0.00 -> 24.6 mm, vias 0 -> 3
- net VDD: track 0.00 -> 18.9 mm, vias 0 -> 7
- net GND: track 0.00 -> 16.8 mm, vias 0 -> 19
- net INT2: track 0.00 -> 9.98 mm, vias 0 -> 2
- net INT1: track 0.00 -> 8.86 mm, vias 0 -> 2
- net Net-(U1-XL2/P0.01): track 0.00 -> 8.81 mm
- net Net-(U1-XL1/P0.00): track 0.00 -> 8.69 mm
- net Net-(AE1-FEED): track 0.00 -> 8.05 mm
- net Net-(U1-XC1): track 0.00 -> 7.98 mm
- net Net-(U1-XC2): track 0.00 -> 7.32 mm
- net SCL: track 0.00 -> 6.32 mm
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- added copper zone on B.Cu, net GND
- added copper zone on F.Cu, net GND
- added copper zone on In1.Cu, net GND
- added copper zone on In2.Cu, net VDD
Other:
- board outline added: 10 x 60 mm

Commit message: Smaller, graphics
Parts:
- added kibuzzard-64E666A5: G***, kibuzzard-64E666A5, F.Cu at (56.4, 90.0)
- added kibuzzard-64E666BF: G***, kibuzzard-64E666BF, F.Cu at (56.4, 87.6)
- added kibuzzard-64E666C8: G***, kibuzzard-64E666C8, F.Cu at (56.4, 85.1)
- added kibuzzard-64E666DB: G***, kibuzzard-64E666DB, F.Cu at (56.4, 82.5)
- added kibuzzard-64E666EE: G***, kibuzzard-64E666EE, F.Cu at (56.4, 79.9)
- added kibuzzard-64E66706: G***, kibuzzard-64E66706, F.Cu at (56.4, 77.6)
- added kibuzzard-64E667F3: G***, kibuzzard-64E667F3, F.Cu at (55.0, 122.1)
- added kibuzzard-64E66855: G***, kibuzzard-64E66855, B.Cu at (55.0, 121.0)
- added kibuzzard-64E668FF: G***, kibuzzard-64E668FF, F.Cu at (52.7, 134.7)
- added kibuzzard-64E66915: G***, kibuzzard-64E66915, F.Cu at (57.5, 134.7)
- added kibuzzard-64E66B38: G***, kibuzzard-64E66B38, B.Cu at (55.0, 123.0)
- added kibuzzard-64E66C17: G***, kibuzzard-64E66C17, F.Cu at (53.0, 78.0)
- moved TP6 51.5 mm to (58.4, 77.5), turned to 90 degrees
- moved H2 16.8 mm to (55.0, 130.2)
- moved S2 4.54 mm to (54.7, 125.0)
- moved BT1 2.49 mm to (52.7, 134.7)
- moved TP2 1.27 mm to (58.4, 87.6)
- moved TP1 1.27 mm to (58.4, 90.2)
- moved TP3 1.27 mm to (58.4, 85.1)
- moved TP4 1.27 mm to (58.4, 82.5)
- moved TP5 1.27 mm to (58.4, 80.0)
Routing:
- net BTN_A: track 29.1 -> 23.4 mm
- net RST: track 34.8 -> 36.3 mm
- net SWDCLK: track 25.9 -> 26.9 mm
- net SWDIO: track 29.3 -> 30.2 mm
Other:
- board size 10 x 60 mm -> 10 x 61 mm
